File: cad_files/mm1a.sch (KiCad schematic (older format))
At the start: 38 parts, among them J1 RELAY, J1a SPST, J2 RELAY, J2a SPST, J3 RELAY, J3a SPST, K1 SPST, K2 DUAL_SWITCH_INV, K3 SPST, K4 SPST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

Commit message: #170914
Parts:
- removed La1: Glimm, VALVE-MINI_P, symbol STABI
- removed La2, La3, La4: glimm, VALVE-MINI_P, symbol STABI
- added La1, La2, La3, La4: GLIMM, glimm, symbol GLIMM
- D1, D2: value D237 -> 1N4001
Connections:
- net labels removed: +12V, GND
- wire segments 97 -> 106
Other:
- note added: "Kézi / Automata"
- note added: "Világítás\nSzellőzés\nFűtés"
- note removed: "Kézi / Automata\nVilágítás\nSzellőztetés\nFűtés"
- moved on the sheet: Cs1, D3, D4, D5, IK1, IK2, J1, J2, J3, K2A, K2B, K3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

Commit message: #171210
Parts:
- removed IK1, IK2: SPST, ~, symbol SPST
- added K6, K7: TSGM1, ~, symbol TIMER
- J1, J2: value RELAY -> 40.52
- J3: value RELAY -> 60.13.9.012.0040
- La1, La2, La3, La4: value GLIMM -> TN-0,3
Connections:
- net labels removed: HT
- wire segments 106 -> 113
Other:
- note added: "Folyamatos / Automata"
- note added: "Világítás\n\nSzellőzés\n\nFűtés"
- note removed: "Időkapcsoló tápfeszültség\n230V AC"
- note removed: "Kézi / Automata"
- note removed: "Világítás\nSzellőzés\nFűtés"
- moved on the sheet: D10, D11, D6, D7, D8, D9, J1, J2, J3, K3, K4, K5

Commit message: 
Parts:
- added D? (x3): D237, ~, symbol DIODE
- added K? (x3): SPST, ~, symbol SPST
Connections:
- net labels added: AGND
- wire segments 113 -> 152
Other:
- note added: "+12V"
- note added: "230V AC L"
- note added: "230V AC N"
- moved on the sheet: Cs1, Cs2, D1, D10, D11, D2, D3, D4, D5, D6, D7, D8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

Commit message: #180514
Parts:
- removed D? (x2): D237, ~, symbol DIODE
- removed K2: DUAL_SWITCH_INV, ~, symbol DUAL_SWITCH_INV
- added D13, D14: 1N4001, ~, symbol DIODE
- added K2a, K2b: SWITCH_INV, ~, symbol SWITCH_INV
- D12: renamed from D?; value D237 -> 1N4001
- gave numbers to parts that had none: 3
- renumbered K1 to K1a
Other:
- note added: "Belső\n\n |\n\nKülső"
- note added: "Szellőztetés - Időzítő ki"
- note added: "Vezérlés"
- note added: "Világítás - Időzítő ki"
- note removed: "Vezérlés\n\nBelső\nKülső"
Changed lines of the file:
@@
 Sheet 1 1
 Title "MM1A gombatermeszto automatika"
-Date "6 may 2018"
+Date "14 may 2018"
 Rev "1.0"
 Comp "Pozsár Zsolt"
@@
 $EndComp
 $Comp
-L DUAL_SWITCH_INV K2
-U 1 1 59ABDD40
-P 2200 4750
-F 0 "K2" H 2000 4900 50  0000 C CNN
-F 1 "DUAL_SWITCH_INV" H 2050 4600 50  0001 C CNN
-F 2 "~" H 2200 4750 60  0000 C CNN
-F 3 "~" H 2200 4750 60  0000 C CNN
-	1    2200 4750
-	1    0    0    -1
-$EndComp
-$Comp
-L DUAL_SWITCH_INV K2
-U 2 1 59ABDD4D
-P 2200 6000
-F 0 "K2" H 2000 6150 50  0000 C CNN
-F 1 "DUAL_SWITCH_INV" H 2050 5850 50  0001 C CNN
-F 2 "~" H 2200 6000 60  0000 C CNN
-F 3 "~" H 2200 6000 60  0000 C CNN
-	2    2200 6000
-	1    0    0    -1
-$EndComp
-$Comp
 L RELAY J3
 U 1 1 59ABE13F
 P 6250 4650
 F 0 "J3" H 6425 4750 60  0000 C CNN
-F 1 "60.13.9.012.0040" H 6150 5150 60  0000 C CNN
+F 1 "60.13.9.012.0040" H 6150 5050 60  0000 C CNN
 F 2 "" H 6250 4650 60  0000 C CNN
 F 3 "" H 6250 4650 60  0000 C CNN
@@
 U 1 1 59ABE2AA
 P 2500 2300
-F 0 "R1" H 2400 2200 40  0000 C CNN
+F 0 "R1" H 2350 2200 40  0000 C CNN
 F 1 "56k" H 2650 2400 40  0000 C CNN
 F 2 "~" V 2430 2300 30  0000 C CNN
 F 3 "~" H 2500 2300 30  0000 C CNN
 	1    2500 2300
-	1    0    0    -1
+	1    0    0    1
 $EndComp
 $Comp
@@
 $EndComp
 $Comp
-L SPST K1
+L SPST K1a
 U 1 1 59ABF12B
 P 7300 5000
-F 0 "K1" H 7300 4850 70  0000 C CNN
+F 0 "K1a" H 7300 5200 70  0000 C CNN
 F 1 "SPST" H 7300 4900 70  0001 C CNN
 F 2 "~" H 7300 5000 60  0000 C CNN
@@
 	1    0    0    -1
 $EndComp
-Text Notes 1850 1600 0    60   ~ 0
+Text Notes 1950 1650 0    60   ~ 0
 Hálózat
 $Comp
@@
 Text Notes 7350 6800 0    60   ~ 0
 Hálózat / Kimenetek
-Text Notes 1400 5300 0    60   ~ 0
-Vezérlés\n\nBelső\nKülső
-Text Notes 5200 7250 0    60   ~ 0
+Text Notes 2100 6350 0    60   ~ 0
+Vezérlés
+Text Notes 6200 6950 1    60   ~ 0
 Folyamatos / Automata
 $Comp
@@
 	0    -1   -1   0
 $EndComp
-Text Notes 5550 7100 1    60   ~ 0
+Text Notes 5550 7600 1    60   ~ 0
 Világítás\n\nSzellőzés\n\nFűtés
 $Comp
@@
 P 4250 6450
 F 0 "K6" V 4450 6600 60  0000 C CNN
-F 1 "TSGM1" V 4450 6250 60  0000 C CNN
+F 1 "TSGM1" V 3500 6450 60  0000 C CNN
 F 2 "~" H 4250 6450 60  0000 C CNN
 F 3 "~" H 4250 6450 60  0000 C CNN
@@
 U 1 1 5A2D0CAF
 P 4600 6850
-F 0 "K7" V 4400 7000 60  0000 C CNN
-F 1 "TSGM1" V 4400 6650 60  0000 C CNN
+F 0 "K7" V 4800 7000 60  0000 C CNN
+F 1 "TSGM1" V 4250 6850 60  0000 C CNN
 F 2 "~" H 4600 6850 60  0000 C CNN
 F 3 "~" H 4600 6850 60  0000 C CNN
@@
 	4600 5200 4600 5150
 $Comp
-L SPST K?
+L SPST K8
 U 1 1 5AEF44AE
 P 4250 5700
-F 0 "K?" H 4100 5800 50  0000 C CNN
+F 0 "K8" H 4100 5800 50  0000 C CNN
 F 1 "SPST" H 4250 5600 70  0001 C CNN
 F 2 "~" H 4250 5700 60  0000 C CNN
@@
 $EndComp
 $Comp
-L SPST K?
+L SPST K9
 U 1 1 5AEF44B4
 P 4600 5700
-F 0 "K?" H 4450 5800 50  0000 C CNN
+F 0 "K9" H 4450 5800 50  0000 C CNN
 F 1 "SPST" H 4600 5600 70  0001 C CNN
 F 2 "~" H 4600 5700 60  0000 C CNN
@@
 $EndComp
 $Comp
-L SPST K?
+L SPST K1b
 U 1 1 5AEF44C4
 P 7500 5000
-F 0 "K?" H 7500 4850 70  0000 C CNN
+F 0 "K1b" H 7500 4850 70  0000 C CNN
 F 1 "SPST" H 7500 4900 70  0001 C CNN
 F 2 "~" H 7500 5000 60  0000 C CNN
@@
 P 5300 2250
 F 0 "#PWR?" H 5300 2250 40  0001 C CNN
-F 1 "AGND" H 5300 2180 50  0000 C CNN
+F 1 "AGND" H 5300 2180 50  0001 C CNN
 F 2 "" H 5300 2250 60  0000 C CNN
 F 3 "" H 5300 2250 60  0000 C CNN
@@
 P 1500 6250
 F 0 "#PWR?" H 1500 6250 40  0001 C CNN
-F 1 "AGND" H 1500 6180 50  0000 C CNN
+F 1 "AGND" H 1500 6180 50  0001 C CNN
 F 2 "" H 1500 6250 60  0000 C CNN
 F 3 "" H 1500 6250 60  0000 C CNN
@@
 $EndComp
 $Comp
-L DIODE D?
+L DIODE D12
 U 1 1 5AEF50CE
 P 5500 3350
-F 0 "D?" H 5450 3450 40  0000 C CNN
-F 1 "D237" H 5650 3450 40  0000 C CNN
+F 0 "D12" H 5600 3450 40  0000 C CNN
+F 1 "1N4001" H 5400 3250 40  0000 C CNN
 F 2 "~" H 5500 3350 60  0000 C CNN
 F 3 "~" H 5500 3350 60  0000 C CNN
@@
 	0    -1   1    0
 $EndComp
-$Comp
-L DIODE D?
-U 1 1 5AEF50D4
+Wire Wire Line
+	5500 3150 5500 3050
+Wire Wire Line
+	5500 3050 5700 3050
+Wire Wire Line
+	5700 3050 5900 3050
+Wire Wire Line
+	5900 3050 6550 3050
+Connection ~ 6550 3650
+Wire Wire Line
+	5700 3150 5700 3050
+Connection ~ 5700 3050
+Wire Wire Line
+	5900 3050 5900 3150
+Connection ~ 5900 3050
+$Comp
+L AGND #PWR?
+U 1 1 5AEF5575
+P 6550 4900
+F 0 "#PWR?" H 6550 4900 40  0001 C CNN
+F 1 "AGND" H 6550 4830 50  0001 C CNN
+F 2 "" H 6550 4900 60  0000 C CNN
+F 3 "" H 6550 4900 60  0000 C CNN
+	1    6550 4900
+	1    0    0    -1
+$EndComp
+Text Notes 6750 5600 0    60   ~ 0
+Hálózat
+Wire Notes Line
+	7300 5000 7400 5000
+Text Notes 3100 3050 0    60   ~ 0
++12V
+Text Notes 6250 2600 0    60   ~ 0
+230V AC L
+Text Notes 6250 2900 0    60   ~ 0
+230V AC N
+$Comp
+L DIODE D13
+U 1 1 5AF9AE8A
 P 5700 3350
-F 0 "D?" H 5650 3450 40  0000 C CNN
-F 1 "D237" H 5850 3450 40  0000 C CNN
+F 0 "D13" H 5800 3450 40  0000 C CNN
+F 1 "1N4001" H 5600 3250 40  0000 C CNN
 F 2 "~" H 5700 3350 60  0000 C CNN
 F 3 "~" H 5700 3350 60  0000 C CNN
@@
 $EndComp
 $Comp
-L DIODE D?
-U 1 1 5AEF50DA
+L DIODE D14
+U 1 1 5AF9AE90
 P 5900 3350
-F 0 "D?" H 5850 3450 40  0000 C CNN
-F 1 "D237" H 6050 3450 40  0000 C CNN
+F 0 "D14" H 6000 3450 40  0000 C CNN
+F 1 "1N4001" H 5800 3250 40  0000 C CNN
 F 2 "~" H 5900 3350 60  0000 C CNN
 F 3 "~" H 5900 3350 60  0000 C CNN
@@
 	0    -1   1    0
 $EndComp
-Wire Wire Line
-	5500 3150 5500 3050
-Wire Wire Line
-	5500 3050 5700 3050
-Wire Wire Line
-	5700 3050 5900 3050
-Wire Wire Line
-	5900 3050 6550 3050
-Connection ~ 6550 3650
-Wire Wire Line
-	5700 3150 5700 3050
-Connection ~ 5700 3050
-Wire Wire Line
-	5900 3050 5900 3150
-Connection ~ 5900 3050
-$Comp
-L AGND #PWR?
-U 1 1 5AEF5575
-P 6550 4900
-F 0 "#PWR?" H 6550 4900 40  0001 C CNN
-F 1 "AGND" H 6550 4830 50  0000 C CNN
-F 2 "" H 6550 4900 60  0000 C CNN
-F 3 "" H 6550 4900 60  0000 C CNN
-	1    6550 4900
-	1    0    0    -1
-$EndComp
-Text Notes 6750 5600 0    60   ~ 0
-Hálózat
-Wire Notes Line
-	7300 5000 7400 5000
-Text Notes 3100 3000 0    60   ~ 0
-+12V
-Text Notes 6200 2550 0    60   ~ 0
-230V AC L
-Text Notes 6200 2950 0    60   ~ 0
-230V AC N
+$Comp
+L SWITCH_INV K2b
+U 1 1 5AF9AF2F
+P 2200 6000
+F 0 "K2b" H 2000 6150 50  0000 C CNN
+F 1 "SWITCH_INV" H 2050 5850 50  0001 C CNN
+F 2 "~" H 2200 6000 60  0000 C CNN
+F 3 "~" H 2200 6000 60  0000 C CNN
+	1    2200 6000
+	1    0    0    -1
+$EndComp
+$Comp
+L SWITCH_INV K2a
+U 1 1 5AF9AF3C
+P 2200 4750
+F 0 "K2a" H 2000 4900 50  0000 C CNN
+F 1 "SWITCH_INV" H 2050 4600 50  0001 C CNN
+F 2 "~" H 2200 4750 60  0000 C CNN
+F 3 "~" H 2200 4750 60  0000 C CNN
+	1    2200 4750
+	1    0    0    -1
+$EndComp
+Text Notes 1800 5200 0    60   ~ 0
+Belső\n\n  |\n\nKülső
+Text Notes 4800 6200 1    60   ~ 0
+Szellőztetés - Időzítő ki
+Text Notes 4075 6050 1    60   ~ 0
+Világítás - Időzítő ki
 $EndSCHEMATC

Commit message: #181223
Parts:
- B1, B2, B3: symbol FUSE-EU -> Fuse-EU
- La1, La2, La3, La4: symbol GLIMM -> glimm
- R1, R2, R3, R4: symbol R -> R-RESCUE-mm1a
Connections:
- net labels added: GNDD
- net labels removed: AGND
Other:
- moved on the sheet: Cs2, D10, D11, D3, D4, D5, D6, D7, D8, D9, J1a, J2a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
